File: Sipariş/Mergen Telemetri + Ateşleme.brd (EAGLE design)
At the start: 53.6 x 90.7 mm, 81 parts, among them J2 U.FL, Q2 IRLML6344TRPBF, Q3 IRLML6344TRPBF, U1 STM32F401CCU6UFQFPN-48_7X7X0P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, U2 ADXL345BCCZ, U3 LPS22HB, U4 L86, U6 AMS1117-3.3, U7 AMS1117-3.3, Y1 ABM3B-26.000MHZ-10-1-U-T

Commit message: LOGO was uploaded
Parts:
- moved SG1 0.56 mm to (47.8, 32.9)
Other:
- board text added: "09.03.2021"
- board text removed: "MERGEN 09.03.2021"
