File: telemetry/STM32F302C8T6/STM32F302C8T6/1206/Mergen Telemetri + Ateşleme.sch (EAGLE design)
At the start: 91 parts, among them J2 U.FL, Q2 IRLML6344TRPBF, Q3 IRLML6344TRPBF, U2 BMP280, U3 MPU-6050, U4 L86, U6 AMS1117-3.3, U7 AMS1117-3.3, U8 STM32F302C8T6, X1 JST-XH-04-PIN-LONG-PAD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

Commit message: NMOS trace was be expanded and creating 1206 package version was tried
Parts:
- C10: value 4.7uF -> 1.0uF; device SparkFun-Capacitors:1.0UF-0603-16V-10% -> SparkFun-Capacitors:1.0UF-1206-50V-10%
- C11, C12, C13, C16, C27, C3, C4, C5, C8, C9: value 100nF -> 1.0uF; device SparkFun-Capacitors:1.0UF-0603-16V-10% -> SparkFun-Capacitors:1.0UF-1206-50V-10%
- C14: value 10nF -> 1.0uF; device SparkFun-Capacitors:1.0UF-0603-16V-10% -> SparkFun-Capacitors:1.0UF-1206-50V-10%
- C15, C19: value 25pF -> 1.0uF; device SparkFun-Capacitors:1.0UF-0603-16V-10% -> SparkFun-Capacitors:1.0UF-1206-50V-10%
- C18, C21, C22, C23, C30, C31, C32: value 0.1uF -> 1.0uF; device SparkFun-Capacitors:1.0UF-0603-16V-10% -> SparkFun-Capacitors:1.0UF-1206-50V-10%
- C20: value 2.2nF -> 1.0uF; device SparkFun-Capacitors:1.0UF-0603-16V-10% -> SparkFun-Capacitors:1.0UF-1206-50V-10%
- D1, D6, D7, D8, D9: device SparkFun-LED:LED0603 -> SparkFun-LED:LED1206
- F1, F3: device SparkFun-Fuses:PPTC_HALF-AMP -> adafruit:PTCFUSE-1206
- L2: value BLM15HB221SN1 -> (none); device inductors:BLM15HB221SN1 -> 52101-101-REV-A_v16:RC-MASTER-SMD_FB_1206MP
- R1, R11, R2, R24, R25, R28, R8: value 10k -> 10; device SparkFun-Resistors:1KOHM-0603-1/10W-1% -> SparkFun-Resistors:10OHM-1206-1/4W-1%
- R10, R26, R6: value 3k3 -> 10; device SparkFun-Resistors:1KOHM-0603-1/10W-1% -> SparkFun-Resistors:10OHM-1206-1/4W-1%
- R16, R27: value 1k -> 10; device SparkFun-Resistors:1KOHM-0603-1/10W-1% -> SparkFun-Resistors:10OHM-1206-1/4W-1%
- R17: value 1k5 -> 10; device SparkFun-Resistors:1KOHM-0603-1/10W-1% -> SparkFun-Resistors:10OHM-1206-1/4W-1%
- R18, R19, R20, R29, R9: value 4k7 -> 10; device SparkFun-Resistors:1KOHM-0603-1/10W-1% -> SparkFun-Resistors:10OHM-1206-1/4W-1%
- R21: value 470 -> 10; device SparkFun-Resistors:1KOHM-0603-1/10W-1% -> SparkFun-Resistors:10OHM-1206-1/4W-1%
- R22, R23: value 680 -> 10; device SparkFun-Resistors:1KOHM-0603-1/10W-1% -> SparkFun-Resistors:10OHM-1206-1/4W-1%
- R3: value 100 -> 10; device SparkFun-Resistors:1KOHM-0603-1/10W-1% -> SparkFun-Resistors:10OHM-1206-1/4W-1%
- R30, R4: value 20 -> 10; device SparkFun-Resistors:1KOHM-0603-1/10W-1% -> SparkFun-Resistors:10OHM-1206-1/4W-1%
- R5: value 0 -> 10; device SparkFun-Resistors:1KOHM-0603-1/10W-1% -> SparkFun-Resistors:10OHM-1206-1/4W-1%
- R7: value 220 -> 10; device SparkFun-Resistors:1KOHM-0603-1/10W-1% -> SparkFun-Resistors:10OHM-1206-1/4W-1%
- VDDA3: value 1uF -> 1.0uF; device SparkFun-Capacitors:0.1UF-0603-25V-(+80/-20%) -> SparkFun-Capacitors:1.0UF-1206-50V-10%
- VDDA4: value 100nF -> 1.0uF; device SparkFun-Capacitors:0.1UF-0603-25V-(+80/-20%) -> SparkFun-Capacitors:1.0UF-1206-50V-10%
