File: telemetry/STM32F302C8T6/STM32F302C8T6/REV1.0/Mergen Telemetri + Ateşleme.sch (EAGLE design)
At the start: 91 parts, among them J2 U.FL, Q2 IRLML6344TRPBF, Q3 IRLML6344TRPBF, U2 BMP280, U3 MPU-6050, U4 L86, U6 AMS1117-3.3, U7 AMS1117-3.3, U8 STM32F302C8T6, X1 JST-XH-04-PIN-LONG-PAD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

Commit message: Update was unsuccesfull
Parts:
- C25, C28: device SparkFun-Capacitors:47UF-POLAR-EIA3528-10V-10% -> SparkFun-Capacitors:10UF-POLAR-EIA3216-16V-10%(TANT)
- L2: value BLM15HB221SN1 -> (none); device inductors:BLM15HB221SN1 -> 52101-101-REV-A_v16:RC-MASTER-SMD_FB_0805MP
- R30, R4: value 20 -> 22
Other:
- moved on the sheet: B2, C25, C27, C28, C5, D4, R16
