File: STM32F302C8T6/Mergen Telemetri + Ateşleme.sch (EAGLE design)
At the start: 91 parts, among them J2 U.FL, Q2 IRLML6344TRPBF, Q3 IRLML6344TRPBF, U2 BMP280, U3 MPU-6050, U4 L86, U6 AMS1117-3.3, U7 AMS1117-3.3, U8 STM32F302C8T6, X1 JST-XH-04-PIN-LONG-PAD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

Commit message: 5V lineer regülator was added for ignition outputs
Parts:
- added C1, C24: 22uF, SparkFun-Capacitors:47UF-POLAR-EIA3528-10V-10%
- added C33, C34: 100nF, SparkFun-Capacitors:1.0UF-0603-16V-10%
- added D10: (no value), SparkFun-LED:LED0603
- added D5: B5819W, Diode:SCHOTTKY_MBR0520LT1GDO-219
- added R12: 1k5, SparkFun-Resistors:1KOHM-0603-1/10W-1%
- added U1: AMS1117-3.3, AMS1117-3.3:AMS1117-3.3
Connections:
- new net HT3: U1.HT
- new net N$23: C1.+, C33.1, D5.C, U1.VIN
- new net N$25: D10.A, R12.1
- new net VOUT: APOGEE.2, C24.+, C34.1, MAIN.1, R12.2, U1.VOUT
- net GND: now also C1.-, C24.-, C33.2, C34.2, D10.C, U1.ADJ
- net VCC: now also D5.A; no longer APOGEE.2, MAIN.1

Commit message: Regulator name was changed as 5.0
Parts:
- U1, U7: value AMS1117-3.3 -> AMS1117-5.0
Changed lines of the file:
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@@
 <part name="GND27" library="supply1" library_urn="urn:adsk.eagle:library:371" deviceset="GND" device=""/>
 <part name="GND30" library="supply1" library_urn="urn:adsk.eagle:library:371" deviceset="GND" device=""/>
-<part name="U7" library="AMS1117-3.3" library_urn="urn:adsk.eagle:library:27162810" deviceset="AMS1117-3.3" device="" package3d_urn="urn:adsk.eagle:package:27162813/2"/>
+<part name="U7" library="AMS1117-3.3" library_urn="urn:adsk.eagle:library:27162810" deviceset="AMS1117-3.3" device="" package3d_urn="urn:adsk.eagle:package:27162813/2" value="AMS1117-5.0"/>
 <part name="GND36" library="supply1" library_urn="urn:adsk.eagle:library:371" deviceset="GND" device=""/>
 <part name="U6" library="AMS1117-3.3" library_urn="urn:adsk.eagle:library:27162810" deviceset="AMS1117-3.3" device="" package3d_urn="urn:adsk.eagle:package:27162813/2"/>
@@
 <part name="D5" library="Diode" library_urn="urn:adsk.eagle:library:16378169" deviceset="SCHOTTKY_" device="DO-219" package3d_urn="urn:adsk.eagle:package:9427153/2" technology="MBR0520LT1G" value="B5819W"/>
 <part name="P+2" library="supply1" library_urn="urn:adsk.eagle:library:371" deviceset="VCC" device="" value="8.4V"/>
-<part name="U1" library="AMS1117-3.3" library_urn="urn:adsk.eagle:library:27162810" deviceset="AMS1117-3.3" device="" package3d_urn="urn:adsk.eagle:package:27162813/2"/>
+<part name="U1" library="AMS1117-3.3" library_urn="urn:adsk.eagle:library:27162810" deviceset="AMS1117-3.3" device="" package3d_urn="urn:adsk.eagle:package:27162813/2" value="AMS1117-5.0"/>
 <part name="GND2" library="supply1" library_urn="urn:adsk.eagle:library:371" deviceset="GND" device=""/>
 <part name="D10" library="SparkFun-LED" library_urn="urn:adsk.eagle:library:27167846" deviceset="LED" device="0603" package3d_urn="urn:adsk.eagle:package:27167834/2"/>
